File: hardware/suzie_bot.sch (EAGLE design)
At the start: 24 parts, among them IC1 LT1529CT33, IC2 L9637DDIP-ADAPTED, Y1 14.7456, Y2 6.0

Commit message: Updating board and schematic.
Connections:
- removed net N$11: U$1.D6, U$4.OFF
- removed net N$34: IC1.!SHDN, U$1.D5
- new net N$10: U$1.A6, U$4.OFF
- new net N$9: IC1.!SHDN, U$1.A7
- net CS-KLINE: now also U$1.A5; no longer U$1.A1
- net N$30: now also U$1.A4; no longer U$1.A7
- net N$33: now also U$1.D3; no longer U$1.A0
- net N$36: now also U$1.D8; no longer U$1.D4
Changed lines of the file:
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@@
 <wire x1="-185.42" y1="193.04" x2="-147.32" y2="193.04" width="0.1524" layer="91"/>
 <wire x1="-147.32" y1="193.04" x2="-76.2" y2="193.04" width="0.1524" layer="91"/>
-<wire x1="-76.2" y1="193.04" x2="63.5" y2="193.04" width="0.1524" layer="91"/>
-<wire x1="63.5" y1="193.04" x2="71.12" y2="198.12" width="0.1524" layer="91"/>
-<wire x1="71.12" y1="198.12" x2="71.12" y2="220.98" width="0.1524" layer="91"/>
-<pinref part="IC1" gate="G$1" pin="OUT"/>
-<wire x1="71.12" y1="220.98" x2="71.12" y2="226.06" width="0.1524" layer="91"/>
-<wire x1="71.12" y1="226.06" x2="58.42" y2="226.06" width="0.1524" layer="91"/>
-<pinref part="IC1" gate="G$1" pin="SENSE"/>
-<wire x1="58.42" y1="220.98" x2="71.12" y2="220.98" width="0.1524" layer="91"/>
-<junction x="71.12" y="220.98"/>
-<wire x1="63.5" y1="193.04" x2="76.2" y2="193.04" width="0.1524" layer="91"/>
-<junction x="63.5" y="193.04"/>
+<wire x1="-76.2" y1="193.04" x2="76.2" y2="193.04" width="0.1524" layer="91"/>
 <wire x1="-78.74" y1="162.56" x2="-76.2" y2="165.1" width="0.1524" layer="91"/>
 <pinref part="U$3" gate="G$1" pin="VCC"/>
@@
 <wire x1="-116.84" y1="149.86" x2="-185.42" y2="149.86" width="0.1524" layer="91"/>
 <junction x="-185.42" y="149.86"/>
+<pinref part="IC1" gate="G$1" pin="OUT"/>
+<wire x1="71.12" y1="226.06" x2="58.42" y2="226.06" width="0.1524" layer="91"/>
+<wire x1="71.12" y1="220.98" x2="71.12" y2="226.06" width="0.1524" layer="91"/>
+<pinref part="IC1" gate="G$1" pin="SENSE"/>
+<wire x1="58.42" y1="220.98" x2="71.12" y2="220.98" width="0.1524" layer="91"/>
+<wire x1="71.12" y1="220.98" x2="76.2" y2="215.9" width="0.1524" layer="91"/>
+<junction x="71.12" y="220.98"/>
+<wire x1="76.2" y1="215.9" x2="76.2" y2="193.04" width="0.1524" layer="91"/>
+<junction x="76.2" y="193.04"/>
 </segment>
 </net>
@@
 <net name="CS-KLINE" class="0">
 <segment>
-<pinref part="U$1" gate="G$1" pin="A1"/>
-<wire x1="15.24" y1="142.24" x2="53.34" y2="142.24" width="0.1524" layer="91"/>
-<wire x1="53.34" y1="142.24" x2="78.74" y2="116.84" width="0.1524" layer="91"/>
-<wire x1="78.74" y1="116.84" x2="152.4" y2="116.84" width="0.1524" layer="91"/>
+<wire x1="53.34" y1="116.84" x2="152.4" y2="116.84" width="0.1524" layer="91"/>
 <wire x1="152.4" y1="116.84" x2="160.02" y2="124.46" width="0.1524" layer="91"/>
 <wire x1="160.02" y1="124.46" x2="160.02" y2="162.56" width="0.1524" layer="91"/>
@@
 <pinref part="U$7" gate="G$1" pin="AO/CS"/>
 <wire x1="149.86" y1="170.18" x2="147.32" y2="167.64" width="0.1524" layer="91"/>
+<pinref part="U$1" gate="G$1" pin="A5"/>
+<wire x1="15.24" y1="152.4" x2="17.78" y2="152.4" width="0.1524" layer="91"/>
+<wire x1="17.78" y1="152.4" x2="53.34" y2="116.84" width="0.1524" layer="91"/>
 </segment>
 </net>
 <net name="N$33" class="0">
 <segment>
-<pinref part="U$1" gate="G$1" pin="A0"/>
-<wire x1="15.24" y1="139.7" x2="33.02" y2="139.7" width="0.1524" layer="91"/>
-<wire x1="33.02" y1="139.7" x2="43.18" y2="129.54" width="0.1524" layer="91"/>
-<wire x1="43.18" y1="129.54" x2="43.18" y2="83.82" width="0.1524" layer="91"/>
-<wire x1="43.18" y1="83.82" x2="35.56" y2="76.2" width="0.1524" layer="91"/>
-<wire x1="35.56" y1="76.2" x2="-53.34" y2="76.2" width="0.1524" layer="91"/>
 <pinref part="U$2" gate="G$1" pin="AO/CS"/>
-<wire x1="-53.34" y1="76.2" x2="-73.66" y2="96.52" width="0.1524" layer="91"/>
-<wire x1="-73.66" y1="96.52" x2="-81.28" y2="96.52" width="0.1524" layer="91"/>
-<wire x1="-81.28" y1="96.52" x2="-88.9" y2="88.9" width="0.1524" layer="91"/>
+<wire x1="-88.9" y1="88.9" x2="-30.48" y2="147.32" width="0.1524" layer="91"/>
+<wire x1="-30.48" y1="147.32" x2="-27.94" y2="147.32" width="0.1524" layer="91"/>
+<wire x1="-27.94" y1="147.32" x2="-20.32" y2="154.94" width="0.1524" layer="91"/>
+<pinref part="U$1" gate="G$1" pin="D3"/>
+<wire x1="-20.32" y1="154.94" x2="-17.78" y2="154.94" width="0.1524" layer="91"/>
 </segment>
 </net>
@@
 <wire x1="114.3" y1="220.98" x2="114.3" y2="215.9" width="0.1524" layer="91"/>
 <wire x1="114.3" y1="215.9" x2="104.14" y2="205.74" width="0.1524" layer="91"/>
-<wire x1="104.14" y1="205.74" x2="63.5" y2="205.74" width="0.1524" layer="91"/>
-<pinref part="U$1" gate="G$1" pin="A7"/>
-<wire x1="63.5" y1="205.74" x2="15.24" y2="157.48" width="0.1524" layer="91"/>
-</segment>
-</net>
-<net name="N$34" class="0">
-<segment>
-<pinref part="IC1" gate="G$1" pin="!SHDN"/>
-<wire x1="33.02" y1="220.98" x2="-5.08" y2="220.98" width="0.1524" layer="91"/>
-<wire x1="-5.08" y1="220.98" x2="-25.4" y2="200.66" width="0.1524" layer="91"/>
-<wire x1="-25.4" y1="200.66" x2="-25.4" y2="152.4" width="0.1524" layer="91"/>
-<wire x1="-25.4" y1="152.4" x2="-22.86" y2="149.86" width="0.1524" layer="91"/>
-<pinref part="U$1" gate="G$1" pin="D5"/>
-<wire x1="-22.86" y1="149.86" x2="-17.78" y2="149.86" width="0.1524" layer="91"/>
+<wire x1="104.14" y1="205.74" x2="73.66" y2="205.74" width="0.1524" layer="91"/>
+<wire x1="73.66" y1="205.74" x2="17.78" y2="149.86" width="0.1524" layer="91"/>
+<pinref part="U$1" gate="G$1" pin="A4"/>
+<wire x1="17.78" y1="149.86" x2="15.24" y2="149.86" width="0.1524" layer="91"/>
 </segment>
 </net>
 <net name="N$36" class="0">
 <segment>
-<pinref part="U$1" gate="G$1" pin="D4"/>
-<wire x1="-17.78" y1="152.4" x2="-20.32" y2="152.4" width="0.1524" layer="91"/>
-<wire x1="-20.32" y1="152.4" x2="-22.86" y2="154.94" width="0.1524" layer="91"/>
-<wire x1="-22.86" y1="154.94" x2="-22.86" y2="200.66" width="0.1524" layer="91"/>
+<wire x1="-22.86" y1="144.78" x2="-22.86" y2="200.66" width="0.1524" layer="91"/>
 <wire x1="-22.86" y1="200.66" x2="-33.02" y2="210.82" width="0.1524" layer="91"/>
 <pinref part="U$11" gate="G$1" pin="P$2"/>
 <wire x1="-33.02" y1="210.82" x2="-38.1" y2="210.82" width="0.1524" layer="91"/>
 <wire x1="-38.1" y1="210.82" x2="-45.72" y2="218.44" width="0.1524" layer="91"/>
+<wire x1="-22.86" y1="144.78" x2="-20.32" y2="142.24" width="0.1524" layer="91"/>
+<pinref part="U$1" gate="G$1" pin="D8"/>
+<wire x1="-20.32" y1="142.24" x2="-17.78" y2="142.24" width="0.1524" layer="91"/>
 </segment>
 </net>
@@
 <wire x1="101.6" y1="279.4" x2="104.14" y2="276.86" width="0.1524" layer="91"/>
 <wire x1="104.14" y1="276.86" x2="104.14" y2="269.24" width="0.1524" layer="91"/>
-</segment>
-</net>
-<net name="N$11" class="0">
-<segment>
-<pinref part="U$4" gate="G$1" pin="OFF"/>
-<wire x1="101.6" y1="274.32" x2="99.06" y2="276.86" width="0.1524" layer="91"/>
-<wire x1="99.06" y1="276.86" x2="93.98" y2="276.86" width="0.1524" layer="91"/>
-<wire x1="101.6" y1="274.32" x2="101.6" y2="264.16" width="0.1524" layer="91"/>
-<wire x1="-27.94" y1="200.66" x2="10.16" y2="238.76" width="0.1524" layer="91"/>
-<wire x1="76.2" y1="238.76" x2="10.16" y2="238.76" width="0.1524" layer="91"/>
-<wire x1="-27.94" y1="200.66" x2="-27.94" y2="152.4" width="0.1524" layer="91"/>
-<wire x1="-27.94" y1="152.4" x2="-22.86" y2="147.32" width="0.1524" layer="91"/>
-<pinref part="U$1" gate="G$1" pin="D6"/>
-<wire x1="-22.86" y1="147.32" x2="-17.78" y2="147.32" width="0.1524" layer="91"/>
-<wire x1="101.6" y1="264.16" x2="76.2" y2="238.76" width="0.1524" layer="91"/>
 </segment>
 </net>
@@
 </segment>
 </net>
+<net name="N$9" class="0">
+<segment>
+<pinref part="IC1" gate="G$1" pin="!SHDN"/>
+<wire x1="33.02" y1="220.98" x2="25.4" y2="213.36" width="0.1524" layer="91"/>
+<wire x1="25.4" y1="213.36" x2="25.4" y2="165.1" width="0.1524" layer="91"/>
+<pinref part="U$1" gate="G$1" pin="A7"/>
+<wire x1="15.24" y1="157.48" x2="17.78" y2="157.48" width="0.1524" layer="91"/>
+<wire x1="25.4" y1="165.1" x2="17.78" y2="157.48" width="0.1524" layer="91"/>
+</segment>
+</net>
+<net name="N$10" class="0">
+<segment>
+<pinref part="U$1" gate="G$1" pin="A6"/>
+<wire x1="15.24" y1="154.94" x2="17.78" y2="154.94" width="0.1524" layer="91"/>
+<wire x1="17.78" y1="154.94" x2="63.5" y2="200.66" width="0.1524" layer="91"/>
+<pinref part="U$4" gate="G$1" pin="OFF"/>
+<wire x1="101.6" y1="274.32" x2="99.06" y2="276.86" width="0.1524" layer="91"/>
+<wire x1="99.06" y1="276.86" x2="93.98" y2="276.86" width="0.1524" layer="91"/>
+<wire x1="101.6" y1="274.32" x2="101.6" y2="264.16" width="0.1524" layer="91"/>
+<wire x1="101.6" y1="264.16" x2="76.2" y2="238.76" width="0.1524" layer="91"/>
+<wire x1="63.5" y1="208.28" x2="76.2" y2="220.98" width="0.1524" layer="91"/>
+<wire x1="76.2" y1="220.98" x2="76.2" y2="238.76" width="0.1524" layer="91"/>
+<wire x1="63.5" y1="200.66" x2="63.5" y2="208.28" width="0.1524" layer="91"/>
+</segment>
+</net>

Commit message: Updating board.
Connections:
- net N$33 renamed CS-GPSWIFI
- net GND: now also U$2.I2C/SPI, U$7.I2C/SPI
Changed lines of the file:
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@@
 </segment>
 </net>
-<net name="N$33" class="0">
+<net name="CS-GPSWIFI" class="0">
 <segment>
 <pinref part="U$2" gate="G$1" pin="AO/CS"/>
-<wire x1="-88.9" y1="88.9" x2="-30.48" y2="147.32" width="0.1524" layer="91"/>
-<wire x1="-30.48" y1="147.32" x2="-27.94" y2="147.32" width="0.1524" layer="91"/>
-<wire x1="-27.94" y1="147.32" x2="-20.32" y2="154.94" width="0.1524" layer="91"/>
+<wire x1="-88.9" y1="88.9" x2="-22.86" y2="154.94" width="0.1524" layer="91"/>
 <pinref part="U$1" gate="G$1" pin="D3"/>
-<wire x1="-20.32" y1="154.94" x2="-17.78" y2="154.94" width="0.1524" layer="91"/>
+<wire x1="-22.86" y1="154.94" x2="-17.78" y2="154.94" width="0.1524" layer="91"/>
 </segment>
 </net>
@@
 <net name="N$36" class="0">
 <segment>
-<wire x1="-22.86" y1="144.78" x2="-22.86" y2="200.66" width="0.1524" layer="91"/>
-<wire x1="-22.86" y1="200.66" x2="-33.02" y2="210.82" width="0.1524" layer="91"/>
 <pinref part="U$11" gate="G$1" pin="P$2"/>
-<wire x1="-33.02" y1="210.82" x2="-38.1" y2="210.82" width="0.1524" layer="91"/>
 <wire x1="-38.1" y1="210.82" x2="-45.72" y2="218.44" width="0.1524" layer="91"/>
-<wire x1="-22.86" y1="144.78" x2="-20.32" y2="142.24" width="0.1524" layer="91"/>
 <pinref part="U$1" gate="G$1" pin="D8"/>
-<wire x1="-20.32" y1="142.24" x2="-17.78" y2="142.24" width="0.1524" layer="91"/>
+<wire x1="-38.1" y1="210.82" x2="-38.1" y2="149.86" width="0.1524" layer="91"/>
+<wire x1="-38.1" y1="149.86" x2="-30.48" y2="142.24" width="0.1524" layer="91"/>
+<wire x1="-30.48" y1="142.24" x2="-17.78" y2="142.24" width="0.1524" layer="91"/>
 </segment>
 </net>
@@
 <net name="N$4" class="0">
 <segment>
-<wire x1="-71.12" y1="165.1" x2="-73.66" y2="167.64" width="0.1524" layer="91"/>
 <pinref part="U$3" gate="G$1" pin="CH_PD"/>
-<wire x1="-73.66" y1="167.64" x2="-88.9" y2="167.64" width="0.1524" layer="91"/>
 <pinref part="U$2" gate="G$1" pin="GPIO7/RIA"/>
-<wire x1="-71.12" y1="165.1" x2="-71.12" y2="78.74" width="0.1524" layer="91"/>
+<wire x1="-71.12" y1="157.48" x2="-71.12" y2="78.74" width="0.1524" layer="91"/>
 <wire x1="-71.12" y1="78.74" x2="-81.28" y2="68.58" width="0.1524" layer="91"/>
+<wire x1="-88.9" y1="167.64" x2="-86.36" y2="165.1" width="0.1524" layer="91"/>
+<wire x1="-86.36" y1="165.1" x2="-78.74" y2="165.1" width="0.1524" layer="91"/>
+<wire x1="-78.74" y1="165.1" x2="-71.12" y2="157.48" width="0.1524" layer="91"/>
 </segment>
 </net>
@@
 <wire x1="83.82" y1="144.78" x2="78.74" y2="149.86" width="0.1524" layer="91"/>
 <pinref part="U$7" gate="G$1" pin="VSS"/>
-<wire x1="116.84" y1="144.78" x2="83.82" y2="144.78" width="0.1524" layer="91"/>
+<wire x1="116.84" y1="144.78" x2="93.98" y2="144.78" width="0.1524" layer="91"/>
+<wire x1="93.98" y1="144.78" x2="83.82" y2="144.78" width="0.1524" layer="91"/>
 <wire x1="78.74" y1="149.86" x2="78.74" y2="185.42" width="0.1524" layer="91"/>
 <junction x="78.74" y="195.58"/>
@@
 <pinref part="5V/GND" gate="G$1" pin="P$2"/>
 <wire x1="160.02" y1="205.74" x2="160.02" y2="299.72" width="0.1524" layer="91"/>
+<pinref part="U$7" gate="G$1" pin="I2C/SPI"/>
+<wire x1="116.84" y1="132.08" x2="106.68" y2="132.08" width="0.1524" layer="91"/>
+<wire x1="106.68" y1="132.08" x2="93.98" y2="144.78" width="0.1524" layer="91"/>
+<junction x="93.98" y="144.78"/>
+<pinref part="U$2" gate="G$1" pin="I2C/SPI"/>
+<wire x1="-129.54" y1="53.34" x2="-139.7" y2="53.34" width="0.1524" layer="91"/>
+<wire x1="-139.7" y1="53.34" x2="-152.4" y2="66.04" width="0.1524" layer="91"/>
+<junction x="-152.4" y="66.04"/>
 </segment>
 </net>
@@
 </sheet>
 </sheets>
+<errors>
+</errors>
 </schematic>
 </drawing>
+<compatibility>
+<note version="6.3" minversion="6.2.2" severity="warning">
+Since Version 6.2.2 text objects can contain more than one line,
+which will not be processed correctly with this version.
+</note>
+</compatibility>
 </eagle>

Commit message: SMD-ized;  pre-autorouting.
Parts:
- removed U$10: VOLTAGE-SENSOR, voltage-sensor:VOLTAGE-SENSOR
- removed U$6: LOGIC_LEVEL_CONVERTER, SparkFun-Boards:LOGIC_LEVEL_CONVERTER
- removed U$9: (no value), User-Submitted:LEVEL-CONVERTING-MICROSD
- added C5, C6: 22pF, SparkFun-Passives:CAP0805
- added C7, C8: 0.1uF, SparkFun-Passives:CAP0805
- added GND/3V3/5V: (no value), SparkFun-Connectors:M03PTH
- added IC3: IC_TXB0108-TSSOP-20, dp_devices.v6:IC_TXB0108-TSSOP-20
- added PA0-7, PB0-7, PC0-7, PD0-7: (no value), SparkFun-Connectors:M08
- added PROGRAMMER: (no value), SparkFun-Connectors:M06SILK_FEMALE_PTH
- added R3: 10k, SparkFun-Passives:RESISTOR0805-RES
- added R4: 70k, SparkFun-Passives:RESISTOR0805-RES
- added R5: 50k, SparkFun-Passives:RESISTOR0805-RES
- added U1: ATMEGA1284P-AU, Atmel_By_element14_Batch_1-00:ATMEGA1284P-AU
- added Y3: 16.0, SparkFun-FreqCtrl:CRYSTALHC49US
- C1, C2, C3, C4: device SparkFun-Passives:CAPPTH -> SparkFun-Passives:CAP0805
- IC2: value L9637DDIP-ADAPTED -> L9637D; device st-microelectronics:L9637DDIP-ADAPTED -> st-microelectronics:L9637D
- R1, R2: device SparkFun-Passives:RESISTORPTH-1/6W -> SparkFun-Passives:RESISTOR0805-RES
- U$1: value NANO -> CON_MICROSDHINGED; device Arduino-clone:NANO -> dp_devices.v6:CON_MICROSDHINGED
- U$7: value SC16IS750IPWDIP-24 -> SC16IS750IPW; device nxp-semiconductors:SC16IS750IPWDIP-24 -> nxp-semiconductors:SC16IS750IPW
Connections:
- removed net CS-GPSWIFI: U$1.D3, U$2.AO/CS
- removed net CS-KLINE: U$1.A5, U$7.AO/CS
- removed net CS-MICROSD: U$1.D10, U$9.CS
- removed net MISO: U$1.D12, U$2.-/SO, U$7.-/SO, U$9.DO
- removed net MOSI: U$1.D11, U$2.A1/SI, U$7.A1/SI, U$9.DI
- removed net N$30: U$1.A4, U$10.S
- removed net N$36: U$1.D8, U$11.P$2
- removed net SCLK: U$1.D13, U$2.SCL/SCLK, U$7.SCL/SCLK, U$9.SCK
- new net N$11: IC3.B1, U$2.RXB
- new net N$12: IC3.B2, U$2.TXB
- new net N$13: C8.1, R3.2, U1.~RESET
- new net N$26: IC3.B5, PB0-7.5, U1.PB4(4)
- new net N$27: IC3.A6, U$1.CMD
- new net N$28: IC3.A7, U$1.DAT0
- new net N$PD0/RXD0: PD0-7.1, PROGRAMMER.3, U1.PD0(8)
- new net PA0: PA0-7.1, R4.2, R5.1, U1.PA0(A0)
- new net PA1: PA0-7.2, U1.PA1(A1)
- new net PA2: PA0-7.3, U1.PA2(A2)
- new net PA3: PA0-7.4, U1.PA3(A3)
- new net PA4: PA0-7.5, U1.PA4(A4)
- new net PA5: PA0-7.6, U1.PA5(A5)
- new net PA6: PA0-7.7, U1.PA6(A6)
- new net PA7: PA0-7.8, U1.PA7(A7)
- new net PB0: PB0-7.1, U$11.P$2, U1.PB0(0)
- new net PB1: IC3.OE, PB0-7.2, U1.PB1(1)
- new net PB2: PB0-7.3, U1.PB2(2)
- new net PB3: PB0-7.4, U$2.AO/CS, U1.PB3(3)
- new net PB5/MOSI: IC3.B6, PB0-7.6, U$2.A1/SI, U$7.A1/SI, U1.PB5(5)
- new net PB6/MISO: IC3.B7, PB0-7.7, U$2.-/SO, U$7.-/SO, U1.PB6(6)
- new net PB7/SCLK: IC3.B8, PB0-7.8, U$2.SCL/SCLK, U$7.SCL/SCLK, U1.PB7(7)
- new net PC0: PC0-7.1, U1.PC0(16)
- new net PC1: PC0-7.2, U1.PC1(17)
- new net PC2: PC0-7.3, U1.PC2(18)
- new net PC3: PC0-7.4, U1.PC3(19)
- new net PC4: PC0-7.5, U1.PC4(20)
- new net PC5: PC0-7.6, U1.PC5(21)
- new net PC6: PC0-7.7, U1.PC6(22)
- new net PC7: PC0-7.8, U$7.AO/CS, U1.PC7(23)
- new net PD1/TXD0: PD0-7.2, PROGRAMMER.2, U1.PD1(9)
- new net PD2/RXD1: PD0-7.3, U1.PD2(10)
- new net PD3/TXD1: PD0-7.4, U1.PD3(11)
- new net PD4: PD0-7.5, U1.PD4(12)
- new net PD5: PD0-7.6, U1.PD5(13)
- new net PD6: IC1.!SHDN, PD0-7.7, U1.PD6(14)
- new net PD7: PD0-7.8, U$4.OFF, U1.PD7(15)
- net 12V-OUT: now also R4.1; no longer U$10.VCC
- net 3V3: now also GND/3V3/5V.2, IC3.VA, U$1.VDD; no longer U$6.LV
- net 5V: now also C7.1, GND/3V3/5V.3, IC3.VB, PROGRAMMER.4, R3.1, U1.AVCC, U1.VCC, U1.VCC_2, U1.VCC_3; no longer U$1.RAW, U$6.HV, U$9.VCC
- net EXTGND: now also R5.2; no longer U$10.GND
- net GND: now also C5.2, C6.1, C7.2, GND/3V3/5V.1, IC3.GND, PROGRAMMER.5, PROGRAMMER.6, U$1.VSS, U1.GND, U1.GND_2, U1.GND_3, U1.GND_4; no longer U$1.GND, U$10.I, U$6.GND, U$6.GND@2, U$9.GND
- net N$10: now also C8.2, PROGRAMMER.1; no longer U$1.A6, U$4.OFF
- net N$14: now also IC3.A4, U$5.RX; no longer U$5.TX, U$6.LV_RXO_1
- net N$17: now also IC3.B3, U$2.RXA; no longer U$5.RX, U$6.LV_TXI_1
- net N$22: now also IC3.A3, U$5.TX; no longer U$2.TXB, U$6.HV_RXI_2
- net N$23: now also IC3.B4, U$2.TXA; no longer U$2.RXB, U$6.HV_TXO_2
- net N$24: now also IC3.A5, U$1.CD/DAT3; no longer U$2.TXA, U$6.HV_TXO_1
- net N$25: now also IC3.A8, U$1.CLK; no longer U$2.RXA, U$6.HV_RXI_1
- net N$5: now also IC3.A1; no longer U$6.LV_TXI_2
- net N$6: now also C6.2, U1.XTAL2, Y3.1; no longer U$1.D9, U$9.CD
- net N$8: now also IC3.A2; no longer U$6.LV_RXO_2
- net N$9: now also C5.1, U1.XTAL1, Y3.2; no longer IC1.!SHDN, U$1.A7
Other:
- moved on the sheet: IC1, IC2
