File: hardware/suzie_bot.sch (EAGLE design)
At the start: 37 parts, among them IC1 LT1529CT33, IC2 L9637D, IC3 IC_TXB0108-TSSOP-20, U1 ATMEGA1284P-AU, Y1 14.7456, Y2 6.0, Y3 16.0

Commit message: Fully layed-out.
Connections:
- removed net N$2: U$2.GPIO6/CDA, U$5.ENABLE
- removed net N$25: IC3.A8, U$1.CLK
- removed net N$27: IC3.A6, U$1.CMD
- removed net N$28: IC3.A7, U$1.DAT0
- removed net N$4: U$2.GPIO7/RIA, U$3.CH_PD
- new net MISO3V3: IC3.A7, U$1.DAT0, U$2.-/SO
- new net MOSI3V3: IC3.A6, U$1.CMD, U$2.A1/SI
- new net SKCK3V3: IC3.A8, U$1.CLK, U$2.SCL/SCLK
- net 12V-OUT: now also U$4.VOUT1
- net 5V: now also U1.AREF
- net EXTGND: now also U$4.GND1, U$4.GND2, U$4.GND3
- net N$7: now also U$4.VIN1
- net PA0: no longer R4.2, R5.1
- net PA5: now also IC1.!SHDN
- net PA6: now also U$3.CH_PD
- net PA7: now also R4.2, R5.1
- net PB2: now also U$5.ENABLE
- net PB5/MOSI: no longer U$2.A1/SI
- net PB6/MISO: no longer U$2.-/SO
- net PB7/SCLK: no longer U$2.SCL/SCLK
- net PC6: now also U$4.OFF
- net PD6: no longer IC1.!SHDN
- net PD7: no longer U$4.OFF
